File: keyboard.kicad_pcb (KiCad board)
At the start: 2 copper layers, 251.5 x 86.4 mm, 118 parts, among them J1 Conn_01x04_Male, J2 USB_B_Micro, J4 Conn_01x11_Male, K0 KEYSW, K1 KEYSW, K10 KEYSW, K11 KEYSW, K12 KEYSW, K13 KEYSW, K14 KEYSW, K15 KEYSW, K16 KEYSW, K17 KEYSW, K18 KEYSW, K19 KEYSW, K2 KEYSW, K20 KEYSW, K21 KEYSW, K22 KEYSW, K23 KEYSW, K24 KEYSW, K25 KEYSW, K26 KEYSW, K27 KEYSW, K28 KEYSW, K29 KEYSW, K3 KEYSW, K30 KEYSW, K31 KEYSW, K32 KEYSW, K33 KEYSW, K34 KEYSW, K35 KEYSW, K36 KEYSW, K37 KEYSW, K38 KEYSW, K39 KEYSW, K4 KEYSW, K40 KEYSW, K41 KEYSW, K42 KEYSW, K43 KEYSW, K5 KEYSW, K6 KEYSW, K7 KEYSW, K8 KEYSW, K9 KEYSW, U1 AMS1117-3.3, U7 RP2040, U8 W25Q128JVS, Y1 12MHz

Commit message: No microchip, keep it basic
Parts:
- removed C1, C2: 10u, Capacitor_SMD:C_0402_1005Metric
- removed C10, C8: 1u, Capacitor_SMD:C_0402_1005Metric
- removed C11, C12, C13, C16, C3, C4, C5, C6, C7, C9: 100n, Capacitor_SMD:C_0402_1005Metric
- removed C14, C15: 30p, Capacitor_SMD:C_0402_1005Metric
- removed J2: USB_B_Micro, Connector_USB:USB_Micro-B_Amphenol_10103594-0001LF_Horizontal
- removed R4, R5: 27R, Resistor_SMD:R_0402_1005Metric
- removed R6: 1k, Resistor_SMD:R_0402_1005Metric
- removed U1: AMS1117-3.3, Package_TO_SOT_SMD:SOT-223-3_TabPin2
- removed U7: RP2040, RP2040_minimal:RP2040-QFN-56
- removed U8: W25Q128JVS, Package_SO:SOIC-8W_5.3x5.3mm_P1.27mm
- removed Y1: 12MHz, Crystal:Crystal_SMD_3225-4Pin_3.2x2.5mm
- J1, J4: moved to B.Cu
- turned J1 to 180 degrees
- turned J4 to -90 degrees
Routing:
- net Net-(C14-Pad1): track 7.19 -> 0.00 mm
- net GND: track 2.90 -> 0.00 mm

Commit message: Added a bit of text
Other:
- board text added: "phoenix keyboard - (c) 2022 sh0ck & pelrun"
Changed lines of the file:
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@@
   )
   (gr_rect (start 86.36 111.76) (end 337.82 198.12) (layer "Edge.Cuts") (width 0.05) (fill none))
+  (gr_text "phoenix keyboard - (c) 2022 sh0ck & pelrun" (at 289.56 193.04) (layer "F.SilkS")
+    (effects (font (size 2 2) (thickness 0.15) italic))
+  )
   (segment (start 88.9 127) (end 88.9 127.503) (width 0.25) (layer "B.Cu") (net 0))
   (segment (start 104.126 129.78) (end 104.101 129.755) (width 0.25) (layer "B.Cu") (net 1))

Commit message: And reroute a few things, smaller board
Parts:
- removed H3, H4: MountingHole, MountingHole:MountingHole_3.2mm_M3_DIN965
- moved H1 29.7 mm to (323.9, 144.3)
- moved H2 28.3 mm to (99.1, 143.1)
- moved J1 24.1 mm to (111.2, 113.1), turned to 90 degrees
- moved J4 9.62 mm to (119.3, 113.1)
Routing:
- net /Row_1: track 200.8 -> 251.6 mm
- net /Row_2: track 243.4 -> 274.3 mm
- net /Row_3: track 338.7 -> 366.8 mm
- net /Col_9: track 244.9 -> 219.8 mm
- net /Col_10: track 232.7 -> 223.5 mm
- net /Col_3: track 121.0 -> 111.8 mm
- net /Col_1: track 95.5 -> 86.3 mm
- net /Col_2: track 111.9 -> 102.7 mm
- net /Col_6: track 178.3 -> 169.0 mm
- net /Col_5: track 154.1 -> 144.9 mm
- net /Col_8: track 211.1 -> 201.9 mm
- net /Col_7: track 193.5 -> 184.6 mm
- net /Row_0: track 208.2 -> 217.0 mm
- net /Col_4: track 133.6 -> 125.1 mm
- net /Col_0: track 70.9 -> 77.3 mm
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Other:
- board size 251.5 x 86.4 mm -> 233.1 x 83.1 mm
- board text added: "ph0en1x by sh0ckdesign & pelrun - revision 1.0"
- board text removed: "phoenix keyboard - (c) 2022 sh0ck & pelrun"
