File: keyboard.kicad_sch (KiCad schematic)
At the start: 94 parts, among them J1 Conn_01x04_Male, J4 Conn_01x11_Male, K0 KEYSW, K1 KEYSW, K10 KEYSW, K11 KEYSW, K12 KEYSW, K13 KEYSW, K14 KEYSW, K15 KEYSW, K16 KEYSW, K17 KEYSW, K18 KEYSW, K19 KEYSW, K2 KEYSW, K20 KEYSW, K21 KEYSW, K22 KEYSW, K23 KEYSW, K24 KEYSW, K25 KEYSW, K26 KEYSW, K27 KEYSW, K28 KEYSW, K29 KEYSW, K3 KEYSW, K30 KEYSW, K31 KEYSW, K32 KEYSW, K33 KEYSW, K34 KEYSW, K35 KEYSW, K36 KEYSW, K37 KEYSW, K38 KEYSW, K39 KEYSW, K4 KEYSW, K40 KEYSW, K41 KEYSW, K42 KEYSW, K43 KEYSW, K5 KEYSW, K6 KEYSW, K7 KEYSW, K8 KEYSW, K9 KEYSW

Commit message: Hmm
Other:
- removed sheet rp2040

Commit message: Moar changes
Parts:
- removed H3, H4: MountingHole, MountingHole:MountingHole_3.2mm_M3_DIN965, symbol Mechanical:MountingHole
Changed lines of the file:
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@@
-    )
-  )
-  (symbol (lib_id "Mechanical:MountingHole") (at 52.07 220.98 0) (unit 1)
-    (in_bom no) (on_board yes)
-    (property "Reference" "H4" (id 0) (at 54.61 219.8116 0)
-      (effects (font (size 1.27 1.27)) (justify left))
-    )
-    (property "Value" "MountingHole" (id 1) (at 54.61 222.123 0)
-      (effects (font (size 1.27 1.27)) (justify left))
-    )
-    (property "Footprint" "MountingHole:MountingHole_3.2mm_M3_DIN965" (id 2) (at 52.07 220.98 0)
-      (effects (font (size 1.27 1.27)) hide)
-    )
-    (property "Datasheet" "https://datasheet.lcsc.com/lcsc/2201251830_JSMSEMI-1N4007WS_C2687395.pdf" (id 3) (at 52.07 220.98 0)
-      (effects (font (size 1.27 1.27)) hide)
-    )
-  )
-  (symbol (lib_id "Mechanical:MountingHole") (at 52.07 232.41 0) (unit 1)
-    (in_bom no) (on_board yes)
-    (property "Reference" "H3" (id 0) (at 54.61 231.2416 0)
-      (effects (font (size 1.27 1.27)) (justify left))
-    )
-    (property "Value" "MountingHole" (id 1) (at 54.61 233.553 0)
-      (effects (font (size 1.27 1.27)) (justify left))
-    )
-    (property "Footprint" "MountingHole:MountingHole_3.2mm_M3_DIN965" (id 2) (at 52.07 232.41 0)
-      (effects (font (size 1.27 1.27)) hide)
-    )
-    (property "Datasheet" "https://datasheet.lcsc.com/lcsc/2201251830_JSMSEMI-1N4007WS_C2687395.pdf" (id 3) (at 52.07 232.41 0)
-      (effects (font (size 1.27 1.27)) hide)
     )
   )
@@
       (reference "H2") (unit 1) (value "MountingHole") (footprint "MountingHole:MountingHole_3.2mm_M3_DIN965")
     )
-    (path "/00000000-0000-0000-0000-00005e99e1a5"
-      (reference "H3") (unit 1) (value "MountingHole") (footprint "MountingHole:MountingHole_3.2mm_M3_DIN965")
-    )
-    (path "/00000000-0000-0000-0000-00005e99cf54"
-      (reference "H4") (unit 1) (value "MountingHole") (footprint "MountingHole:MountingHole_3.2mm_M3_DIN965")
-    )
     (path "/ab2b0d87-f1e5-451b-abfd-998cd9f101f9"
